Commit message: added camera for vla

File: src/environment/resource/roarm.urdf (robot description, URDF)
Before this commit: robot physics, 11 links, 10 joints
Joints:
- joint L1_to_L2: origin xyz=0 0.041051 0.0534 rpy=0.655391 0 0 -> xyz=0 0.041051 0.05624 rpy=0.655391 0 0
- joint base_to_L1: origin xyz=0 0 0.062 -> xyz=0 0 0.0595
